Commit message: Robot xacro updated to included wheels

File: src/my_robot/urdf/my_robot.xacro (robot description, xacro)
@@ -54,3 +54,65 @@
     </visual>
   </link>
+  <link name='left_wheel'>
+    <inertial>
+      <mass value="5.0"/>
+      <origin xyz="0.0 0 0" rpy=" 0 1.5707 1.5707"/>
+      <inertia
+          ixx="0.1" ixy="0" ixz="0"
+          iyy="0.1" iyz="0"
+          izz="0.1"
+      />
+    </inertial>
+    <collision name='collision'>
+      <origin xyz="0.0 0 0" rpy=" 0 1.5707 1.5707"/>
+      <geometry>
+        <cylinder radius=".1" length=".05"/>
+      </geometry>
+    </collision>
+    <visual name='left_wheel_visual'>
+      <origin xyz="0.0 0 0" rpy=" 0 1.5707 1.5707"/>
+      <geometry>
+        <cylinder radius=".1" length=".05"/>
+      </geometry>
+    </visual>
+  </link>
+    <link name='right_wheel'>
+    <inertial>
+      <mass value="5.0"/>
+      <origin xyz="0.0 0 0" rpy=" 0 1.5707 1.5707"/>
+      <inertia
+          ixx="0.1" ixy="0" ixz="0"
+          iyy="0.1" iyz="0"
+          izz="0.1"
+      />
+    </inertial>
+    <collision name='collision'>
+      <origin xyz="0.0 0 0" rpy=" 0 1.5707 1.5707"/>
+      <geometry>
+        <cylinder radius=".1" length=".05"/>
+      </geometry>
+    </collision>
+    <visual name='right_wheel_visual'>
+      <origin xyz="0.0 0 0" rpy=" 0 1.5707 1.5707"/>
+      <geometry>
+        <cylinder radius=".1" length=".05"/>
+      </geometry>
+    </visual>
+  </link>
+   <joint type="continuous" name="left_wheel_hinge">
+    <origin xyz="0 0.15 0" rpy="0 0 0"/>
+    <child link="left_wheel"/>
+    <parent link="chassis"/>
+    <axis xyz="0 1 0" rpy="0 0 0"/>
+    <limit effort="10000" velocity="1000"/>
+    <dynamics damping="1.0" friction="1.0"/>
+  </joint>
+   <joint type="continuous" name="right_wheel_hinge">
+    <origin xyz="0 -0.15 0" rpy="0 0 0"/>
+    <child link="right_wheel"/>
+    <parent link="chassis"/>
+    <axis xyz="0 1 0" rpy="0 0 0"/>
+    <limit effort="10000" velocity="1000"/>
+    <dynamics damping="1.0" friction="1.0"/>
+  </joint>
 </robot>

Commit message: Camera & Lidar link added

File: src/my_robot/urdf/my_robot.xacro (robot description, xacro)
@@ -116,3 +116,55 @@
     <dynamics damping="1.0" friction="1.0"/>
   </joint>
+   <!-- Camera link -->
+  <link name="camera">
+  <visual>
+    <geometry>
+      <box size="0.05 0.05 0.05"/>
+    </geometry>
+    <origin xyz="0 0 0" rpy="0 0 0"/>
+  </visual>
+  <collision>
+    <geometry>
+      <box size="0.05 0.05 0.05"/>
+    </geometry>
+    <origin xyz="0 0 0" rpy="0 0 0"/>
+  </collision>
+  <inertial>
+    <mass value="0.1"/>
+    <inertia ixx="1e-6" ixy="0" ixz="0" iyy="1e-6" iyz="0" izz="1e-6"/>
+  </inertial>
+  </link>
+  <!-- Camera joint -->
+ <joint name="camera_joint" type="fixed">
+  <axis xyz="0 1 0"/>
+  <origin xyz="0.2 0 0" rpy="0 0 0"/>
+  <parent link="chassis"/>
+  <child link="camera"/>
+ </joint>
+  <!-- Hokuyo lidar sensor link -->
+  <link name="hokuyo">
+  <visual>
+    <geometry>
+      <mesh filename="package://my_robot/meshes/hokuyo.dae"/>
+    </geometry>
+    <origin xyz="0 0 0" rpy="0 0 0"/>
+  </visual>
+  <collision>
+    <geometry>
+      <box size="0.1 0.1 0.1"/>
+    </geometry>
+    <origin xyz="0 0 0" rpy="0 0 0"/>
+  </collision>
+  <inertial>
+    <mass value="1e-5"/>
+    <inertia ixx="1e-6" ixy="0" ixz="0" iyy="1e-6" iyz="0" izz="1e-6"/>
+  </inertial>
+  </link>
+  <!-- Hokuyo lidar sensor joint -->
+  <joint name="hokuyo_joint" type="fixed">
+  <axis xyz="0 1 0"/>
+  <origin xyz="0.15 0 0.1" rpy="0 0 0"/>
+  <parent link="chassis"/>
+  <child link="hokuyo"/>
+  </joint>
 </robot>

Commit message: Comments addressed

File: src/my_robot/urdf/my_robot.xacro (robot description, xacro)
@@ -29,4 +29,7 @@
         <box size=".4 .2 .1"/>
       </geometry>
+      <material name="blue">
+        <color rgba="0 0 1 1"/>
+      </material>
     </visual>
     <collision name='back_caster_collision'>
@@ -41,4 +44,7 @@
         <sphere radius="0.05"/>
       </geometry>
+      <material name="grey">
+        <color rgba="0.5 0.5 0.5 1"/>
+      </material>
     </visual>
     <collision name='front_caster_collision'>
@@ -53,4 +59,7 @@
         <sphere radius="0.05"/>
       </geometry>
+      <material name="grey">
+        <color rgba="0.5 0.5 0.5 1"/>
+      </material>
     </visual>
   </link>
@@ -76,4 +85,7 @@
         <cylinder radius=".1" length=".05"/>
       </geometry>
+      <material name="black">
+        <color rgba="0 0 0 1"/>
+      </material>
     </visual>
   </link>
@@ -99,4 +111,7 @@
         <cylinder radius=".1" length=".05"/>
       </geometry>
+      <material name="black">
+        <color rgba="0 0 0 1"/>
+      </material>
     </visual>
   </link>
@@ -124,4 +139,7 @@
     </geometry>
     <origin xyz="0 0 0" rpy="0 0 0"/>
+    <material name="black">
+      <color rgba="0 0 0 1"/>
+    </material>
   </visual>
   <collision>

Commit message: Color added

File: src/my_robot/urdf/my_robot.xacro (robot description, xacro)
@@ -2,5 +2,5 @@
   <xacro:include filename="$(find my_robot)/urdf/my_robot.gazebo" />
   <link name="robot_footprint"></link>
-  <joint name="robot_footprint_joint" type="fixed">
+  <joint name="robot_footprint" type="fixed">
     <origin xyz="0 0 0" rpy="0 0 0" />
     <parent link="robot_footprint"/>
@@ -187,3 +187,15 @@
   <child link="hokuyo"/>
   </joint>
+    <gazebo reference="left_wheel">
+    <material>Gazebo/Red</material>
+  </gazebo>
+  <gazebo reference="right_wheel">
+    <material>Gazebo/Red</material>
+  </gazebo>
+  <gazebo reference="chassis">
+    <material>Gazebo/Yellow</material>
+  </gazebo>
+  <gazebo reference="camera">
+    <material>Gazebo/Black</material>
+  </gazebo>
 </robot>

Commit message: Robot updated

File: src/my_robot/urdf/my_robot.xacro (robot description, xacro)
@@ -1,6 +1,7 @@
+<?xml version='1.0'?>
 <robot name="my_robot" xmlns:xacro="http://www.ros.org/wiki/xacro">
   <xacro:include filename="$(find my_robot)/urdf/my_robot.gazebo" />
   <link name="robot_footprint"></link>
-  <joint name="robot_footprint" type="fixed">
+  <joint name="robot_footprint_joint" type="fixed">
     <origin xyz="0 0 0" rpy="0 0 0" />
     <parent link="robot_footprint"/>
@@ -13,7 +14,7 @@
       <origin xyz="0.0 0 0" rpy=" 0 0 0"/>
       <inertia
-          ixx="0.1" ixy="0" ixz="0"
-          iyy="0.1" iyz="0"
-          izz="0.1"
+              ixx="0.1" ixy="0" ixz="0"
+              iyy="0.1" iyz="0"
+              izz="0.1"
       />
     </inertial>
@@ -29,7 +30,4 @@
         <box size=".4 .2 .1"/>
       </geometry>
-      <material name="blue">
-        <color rgba="0 0 1 1"/>
-      </material>
     </visual>
     <collision name='back_caster_collision'>
@@ -44,7 +42,4 @@
         <sphere radius="0.05"/>
       </geometry>
-      <material name="grey">
-        <color rgba="0.5 0.5 0.5 1"/>
-      </material>
     </visual>
     <collision name='front_caster_collision'>
@@ -59,63 +54,53 @@
         <sphere radius="0.05"/>
       </geometry>
-      <material name="grey">
-        <color rgba="0.5 0.5 0.5 1"/>
-      </material>
     </visual>
   </link>
-  <link name='left_wheel'>
+  <!-- Add two wheels -->
+  <link name="left_wheel">
     <inertial>
-      <mass value="5.0"/>
-      <origin xyz="0.0 0 0" rpy=" 0 1.5707 1.5707"/>
+      <origin xyz="0 0 0" rpy="0 1.5707 1.5707"/>
+      <mass value="5"/>
       <inertia
-          ixx="0.1" ixy="0" ixz="0"
-          iyy="0.1" iyz="0"
-          izz="0.1"
+              ixx="0.1" ixy="0" ixz="0"
+              iyy="0.1" iyz="0" izz="0.1"
       />
     </inertial>
-    <collision name='collision'>
-      <origin xyz="0.0 0 0" rpy=" 0 1.5707 1.5707"/>
+    <collision>
+      <origin xyz="0 0 0" rpy="0 1.5707 1.5707"/>
       <geometry>
-        <cylinder radius=".1" length=".05"/>
+        <cylinder radius="0.1" length="0.05"/>
       </geometry>
     </collision>
-    <visual name='left_wheel_visual'>
-      <origin xyz="0.0 0 0" rpy=" 0 1.5707 1.5707"/>
+    <visual>
+      <origin xyz="0 0 0" rpy="0 1.5707 1.5707"/>
       <geometry>
-        <cylinder radius=".1" length=".05"/>
+        <cylinder radius="0.1" length="0.05"/>
       </geometry>
-      <material name="black">
-        <color rgba="0 0 0 1"/>
-      </material>
     </visual>
   </link>
-    <link name='right_wheel'>
+  <link name="right_wheel">
     <inertial>
-      <mass value="5.0"/>
-      <origin xyz="0.0 0 0" rpy=" 0 1.5707 1.5707"/>
+      <origin xyz="0 0 0" rpy="0 1.5707 1.5707"/>
+      <mass value="5"/>
       <inertia
-          ixx="0.1" ixy="0" ixz="0"
-          iyy="0.1" iyz="0"
-          izz="0.1"
+              ixx="0.1" ixy="0" ixz="0"
+              iyy="0.1" iyz="0" izz="0.1"
       />
     </inertial>
-    <collision name='collision'>
-      <origin xyz="0.0 0 0" rpy=" 0 1.5707 1.5707"/>
+    <collision>
+      <origin xyz="0 0 0" rpy="0 1.5707 1.5707"/>
       <geometry>
-        <cylinder radius=".1" length=".05"/>
+        <cylinder radius="0.1" length="0.05"/>
       </geometry>
     </collision>
-    <visual name='right_wheel_visual'>
-      <origin xyz="0.0 0 0" rpy=" 0 1.5707 1.5707"/>
+    <visual>
+      <origin xyz="0 0 0" rpy="0 1.5707 1.5707"/>
       <geometry>
-        <cylinder radius=".1" length=".05"/>
+        <cylinder radius="0.1" length="0.05"/>
       </geometry>
-      <material name="black">
-        <color rgba="0 0 0 1"/>
-      </material>
     </visual>
   </link>
-   <joint type="continuous" name="left_wheel_hinge">
-    <origin xyz="0 0.15 0" rpy="0 0 0"/>
+  <joint name="left_wheel_hinge" type="continuous">
+    <origin xyz="0 0.125 0" rpy="0 0 0"/>
     <child link="left_wheel"/>
     <parent link="chassis"/>
@@ -124,6 +109,6 @@
     <dynamics damping="1.0" friction="1.0"/>
   </joint>
-   <joint type="continuous" name="right_wheel_hinge">
-    <origin xyz="0 -0.15 0" rpy="0 0 0"/>
+  <joint name="right_wheel_hinge" type="continuous">
+    <origin xyz="0 -0.125 0" rpy="0 0 0"/>
     <child link="right_wheel"/>
     <parent link="chassis"/>
@@ -132,70 +117,70 @@
     <dynamics damping="1.0" friction="1.0"/>
   </joint>
-   <!-- Camera link -->
+  <!-- Add camera -->
   <link name="camera">
-  <visual>
-    <geometry>
-      <box size="0.05 0.05 0.05"/>
-    </geometry>
-    <origin xyz="0 0 0" rpy="0 0 0"/>
-    <material name="black">
-      <color rgba="0 0 0 1"/>
-    </material>
-  </visual>
-  <collision>
-    <geometry>
-      <box size="0.05 0.05 0.05"/>
-    </geometry>
-    <origin xyz="0 0 0" rpy="0 0 0"/>
-  </collision>
-  <inertial>
-    <mass value="0.1"/>
-    <inertia ixx="1e-6" ixy="0" ixz="0" iyy="1e-6" iyz="0" izz="1e-6"/>
-  </inertial>
+    <origin xyz="0 0 0" rpy="0 0 0" />
+    <inertial>
+      <mass value="0.1"/>
+      <inertia
+              ixx="1e-6" ixy="0" ixz="0"
+              iyy="1e-6" iyz="0" izz="1e-6"
+      />
+    </inertial>
+    <collision>
+      <geometry>
+        <box size="0.05 0.05 0.05"/>
+      </geometry>
+    </collision>
+    <visual>
+      <geometry>
+        <box size="0.05 0.05 0.05"/>
+      </geometry>
+    </visual>
   </link>
-  <!-- Camera joint -->
- <joint name="camera_joint" type="fixed">
-  <axis xyz="0 1 0"/>
-  <origin xyz="0.2 0 0" rpy="0 0 0"/>
-  <parent link="chassis"/>
-  <child link="camera"/>
- </joint>
-  <!-- Hokuyo lidar sensor link -->
+  <joint name="camera_joint" type="fixed">
+    <axis xyz="0 1 0"/>
+    <origin xyz="0.2 0 0" rpy="0 0 0" />
+    <parent link="chassis"/>
+    <child link="camera" />
+  </joint>
+  <!-- Add Lidar -->
   <link name="hokuyo">
-  <visual>
-    <geometry>
-      <mesh filename="package://my_robot/meshes/hokuyo.dae"/>
-    </geometry>
-    <origin xyz="0 0 0" rpy="0 0 0"/>
-  </visual>
-  <collision>
-    <geometry>
-      <box size="0.1 0.1 0.1"/>
-    </geometry>
-    <origin xyz="0 0 0" rpy="0 0 0"/>
-  </collision>
-  <inertial>
-    <mass value="1e-5"/>
-    <inertia ixx="1e-6" ixy="0" ixz="0" iyy="1e-6" iyz="0" izz="1e-6"/>
-  </inertial>
+    <origin xyz="0 0 0" rpy="0 0 0" />
+    <inertial>
+      <mass value="1e-5"/>
+      <inertia
+              ixx="1e-6" ixy="0" ixz="0"
+              iyy="1e-6" iyz="0" izz="1e-6"
+      />
+    </inertial>
+    <collision>
+      <geometry>
+        <box size=".1 .1 .1"/>
+      </geometry>
+    </collision>
+    <visual>
+      <geometry>
+        <mesh filename="package://my_robot/meshes/hokuyo.dae"/>
+      </geometry>
+    </visual>
   </link>
-  <!-- Hokuyo lidar sensor joint -->
   <joint name="hokuyo_joint" type="fixed">
-  <axis xyz="0 1 0"/>
-  <origin xyz="0.15 0 0.1" rpy="0 0 0"/>
-  <parent link="chassis"/>
-  <child link="hokuyo"/>
+    <axis xyz="0 1 0"/>
+    <origin xyz="0.15 0 0.1" rpy="0 0 0" />
+    <parent link="chassis"/>
+    <child link="hokuyo" />
   </joint>
-    <gazebo reference="left_wheel">
+  <!-- Color the components -->
+  <gazebo reference="chassis">
+    <material>Gazebo/Orange</material>
+  </gazebo>
+  <gazebo reference="left_wheel">
+    <material>Gazebo/Green</material>
+  </gazebo>
+  <gazebo reference="right_wheel">
+    <material>Gazebo/Green</material>
+  </gazebo>
+  <gazebo reference="camera">
     <material>Gazebo/Red</material>
   </gazebo>
-  <gazebo reference="right_wheel">
-    <material>Gazebo/Red</material>
-  </gazebo>
-  <gazebo reference="chassis">
-    <material>Gazebo/Yellow</material>
-  </gazebo>
-  <gazebo reference="camera">
-    <material>Gazebo/Black</material>
-  </gazebo>
-</robot>
+ </robot>
